File: printer_mods/Dotdash32/SKR_E3_Mini_V2_Expanders/FanExpander-Lite/FanExpander-Lite.kicad_pcb (KiCad board)
At the start: 2 copper layers, 35.1 x 34.7 mm, 31 parts, among them J1 FAN1_IN, J10 FAN2, J11 V_SELECT3, J12 V_SELECT4, J13 FAN3, J14 FAN4, J2 IO_PassThrough, J3 EXP1_IN, J6 V_SELECT1, J7 V_SELECT2, J9 FAN1, Q1 IRLML6344, Q2 IRLML6344, Q3 IRLML6344

Commit message: feat: init routing of Lite board
Parts:
- turned F3 to 0 degrees
- turned R10 to 0 degrees
Connections:
- J3 pad 1: /FAN2 -> /PASS0
- J3 pad 2: /PASS1 -> /FAN4
- J3 pad 3: /FAN3 -> /PASS1
- J3 pad 5: /FAN4 -> /PASS2
- J3 pad 6: /PASS2 -> /FAN3
- J3 pad 7: /PASS0 -> /PASS3
- J3 pad 8: /PASS3 -> /FAN2
Routing:
- net +5V: track 0.00 -> 51.6 mm
- net +24V: track 0.00 -> 43.4 mm
- net /LED_Drive: track 0.00 -> 36.8 mm
- net /FAN2: track 0.00 -> 34.9 mm, vias 0 -> 1
- net /5V_unFused: track 0.00 -> 31.8 mm, vias 0 -> 1
- net /PASS3: track 0.00 -> 25.3 mm
- net /PASS0: track 0.00 -> 24.9 mm
- net /FAN3: track 0.00 -> 24.3 mm, vias 0 -> 1
- net /PASS2: track 0.00 -> 24.3 mm
- net /PASS1: track 0.00 -> 24.2 mm
- net /FAN4: track 0.00 -> 24.1 mm, vias 0 -> 1
- net /FAN3_Drive: track 0.00 -> 16.4 mm
- net /FAN2_Drive: track 0.00 -> 15.8 mm
- net /FAN4_Drive: track 0.00 -> 15.8 mm
- net /F4V: track 0.00 -> 14.4 mm
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- added copper zone on B.Cu, net GND
- added copper zone on F.Cu, net GND

Commit message: chore: cleanup edges, silkscreen, making pretty
Parts:
- renumbered D3 to D1, D4 to D2, D5 to D3, D6 to D4, F3 to F2, J9 to J1, J10 to J2, J13 to J3, J14 to J4, J3 to J5, J1 to J6, J2 to J7, J6 to JP1, J7 to JP2, J11 to JP3, J12 to JP4, JP2 to JP5, R2 to R1, R3 to R2, R6 to R3, R5 to R4, R7 to R5, R11 to R6, R9 to R7, R12 to R9
Other:
- outline, holes or cut-outs redrawn
- board text added: "5V F1 24V"
- board text added: "5V F2 24V"
- board text added: "5V F3 24V"
- board text added: "5V F4 24V"
- board text added: "Designed by Dotdash32 (JDeW) 12/21"
- board text added: "Fan1 IN"
- board text added: "Fan1 Pass"
- board text added: "Fan2 PB15"
- board text added: "Fan3 PB9"
- board text added: "Fan4 PA15"
- board text added: "GND"
- board text added: "LED EN (over)"
- board text added: "PB8 PA10 PA0 PB5"
- board text added: "SKR E3 Mini Fan Expander Lite 1+3 Volt Select Fans 4 I/O Pins"
