File: printer_mods/Dotdash32/SKR_E3_Mini_V2_Expanders/FanExpander-kicad/_autosave-FanExpander-kicad.sch (KiCad schematic (older format))
At the start: 66 parts, among them J0 FAN0, J1 FAN1, J10 FAN0_IN, J11 HI_PWR_Inputs, J2 FAN2, J3 FAN3, J4 FAN4, J5 FAN5, J6 FAN6, J7 FAN7, J8 EXP1_IN, J9 5V_In, Q1 IRLML6344, Q2 IRLML6344, Q3 IRLML6344, Q4 IRLML6344, Q5 IRLML6344, Q6 IRLML6344, Q7 IRLML6344

Commit message: feat: breakaway layout, using 1mm spacing headers
it works, but its SOOO LOOOONG, going to try again and make it
more compact so I don't feel bad about this long stick in my printer
Parts:
- MH1, MH2: footprint Mounting_Holes:MountingHole_3.2mm_M3 -> Mounting_Holes:MountingHole_3.2mm_M3_Pad
Changed lines of the file:
@@
 F 0 "MH1" V 5204 7300 50  0000 L CNN
 F 1 "MountingHole" V 5295 7300 50  0000 L CNN
-F 2 "Mounting_Holes:MountingHole_3.2mm_M3" H 5250 7150 50  0001 C CNN
+F 2 "Mounting_Holes:MountingHole_3.2mm_M3_Pad" H 5250 7150 50  0001 C CNN
 F 3 "~" H 5250 7150 50  0001 C CNN
 	1    5250 7150
@@
 F 0 "MH2" V 5204 7500 50  0000 L CNN
 F 1 "MountingHole" V 5295 7500 50  0000 L CNN
-F 2 "Mounting_Holes:MountingHole_3.2mm_M3" H 5250 7350 50  0001 C CNN
+F 2 "Mounting_Holes:MountingHole_3.2mm_M3_Pad" H 5250 7350 50  0001 C CNN
 F 3 "~" H 5250 7350 50  0001 C CNN
 	1    5250 7350
@@
 Connection ~ 2250 4850
 $Comp
-L power:GND #PWR?
+L power:GND #PWR0110
 U 1 1 62644B19
 P 5050 7450
-F 0 "#PWR?" H 5050 7200 50  0001 C CNN
+F 0 "#PWR0110" H 5050 7200 50  0001 C CNN
 F 1 "GND" H 5055 7277 50  0000 C CNN
 F 2 "" H 5050 7450 50  0001 C CNN
