File: printer_mods/Dotdash32/SKR_E3_Mini_V2_Expanders/FanExpander-kicad/FanExpander-kicad.kicad_pcb (KiCad board)
At the start: 2 copper layers, 51.8 x 31.9 mm, 71 parts, among them J0 JST-XH2, J1 JST-XH2, J10 JST-XH2, J12 HI_PWR2, J2 JST-XH2, J3 JST-XH2, J4 JST-XH2, J5 JST-XH2, J6 JST-XH2, J7 JST-XH2, J8 EXPx_IN, J9 5V_In, Q1 IRLML6344, Q2 IRLML6344, Q3 IRLML6344, Q4 IRLML6344, Q5 IRLML6344, Q6 IRLML6344, Q7 IRLML6344

Commit message: chore: update FE to Kicad 6, add resistor 3d comps
Other:
- net class Default removed
- net class Power removed
- net class signal removed
